File: EDA/MRBR/Kicad/MRBR/MRBR.sch (KiCad schematic (older format))
At the start: 7 parts, among them SW1 Reset, U1 ESP32-WROOM-32

Commit message: Resume schematics conception
Connections:
- net labels added: CLK_NC, CMD_NC, SD0_NC, SD1_NC, SD2_NC, SD3_NC, S_VN_NC, S_VP_NC
- wire segments 48 -> 56
- no-connect marks 9 -> 8
Changed lines of the file:
@@
 Wire Wire Line
 	4400 1400 4400 1700
-NoConn ~ 3800 3100
-NoConn ~ 3800 3200
-NoConn ~ 3800 3300
-NoConn ~ 3800 3400
-NoConn ~ 3800 3500
-NoConn ~ 3800 3600
-NoConn ~ 3800 2100
-NoConn ~ 3800 2200
-NoConn ~ 3650 3250
+NoConn ~ 3350 2100
+NoConn ~ 3350 2200
 Wire Wire Line
 	3800 1900 3400 1900
@@
 F1 "PSU.sch" 50
 $EndSheet
+Wire Wire Line
+	3800 3100 3350 3100
+Wire Wire Line
+	3350 3200 3800 3200
+Wire Wire Line
+	3350 3300 3800 3300
+Wire Wire Line
+	3350 3400 3800 3400
+Wire Wire Line
+	3350 3500 3800 3500
+Wire Wire Line
+	3350 3600 3800 3600
+NoConn ~ 3350 3100
+NoConn ~ 3350 3200
+NoConn ~ 3350 3300
+NoConn ~ 3350 3400
+NoConn ~ 3350 3500
+NoConn ~ 3350 3600
+Wire Wire Line
+	3800 2100 3350 2100
+Wire Wire Line
+	3350 2200 3800 2200
 Wire Bus Line
 	6350 3400 6350 3600
@@
 Wire Bus Line
 	5450 3600 5450 4300
+Text Label 3450 2100 0    50   ~ 0
+S_VP_NC
+Text Label 3450 2200 0    50   ~ 0
+S_VN_NC
+Text Label 3450 3100 0    50   ~ 0
+SD0_NC
+Text Label 3450 3200 0    50   ~ 0
+SD1_NC
+Text Label 3450 3300 0    50   ~ 0
+SD2_NC
+Text Label 3450 3400 0    50   ~ 0
+SD3_NC
+Text Label 3450 3500 0    50   ~ 0
+CLK_NC
+Text Label 3450 3600 0    50   ~ 0
+CMD_NC
 $EndSCHEMATC
