File: Hardware/Node/Node.kicad_sch (KiCad schematic)
At the start: 0 parts

Commit message: Updated schematic
Other:
- added sheet Power Supply (psu.kicad_sch)
- sheet ESP32 ports: added EMAC_CLK_OUT_180, EMAC_RXD0(RMII), EMAC_RXD1(RMII), EMAC_RX_CRX_DV, EMAC_TXD0(RMII), EMAC_TXD1(RMII), EMAC_TX_EN(RMII), EN, I2C_SCL, I2C_SDA, I2S0_DOUT, I2S0_WS, I2S1_DOUT, I2S1_WS, I2S_SCL, IO0, MDC(RMII), MDIO(RMII), PHY_PWR, UART_RX0, UART_TX0; removed none
Changed lines of the file:
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@@
     (rev "1.0.0")
   )
-  (sheet (at 151.13 41.275) (size 19.685 17.78) (fields_autoplaced)
+  (sheet (at 137.795 80.01) (size 19.685 12.7) (fields_autoplaced)
     (stroke (width 0.1524) (type solid))
     (fill (color 0 0 0 0.0000))
-    (property "Sheetname" "Track Control" (at 151.13 40.5634 0)
+    (property "Sheetname" "Track Control" (at 137.795 79.2984 0)
       (effects (font (size 1.27 1.27)) (justify left bottom))
     )
-    (property "Sheetfile" "track_ctrl.kicad_sch" (at 151.13 59.6396 0)
+    (property "Sheetfile" "track_ctrl.kicad_sch" (at 137.795 93.2946 0)
       (effects (font (size 1.27 1.27)) (justify left top))
     )
@@
     )
   )
-  (sheet (at 67.31 60.96) (size 17.145 27.94) (fields_autoplaced)
+  (sheet (at 78.105 111.76) (size 12.7 3.81) (fields_autoplaced)
     (stroke (width 0.1524) (type solid))
     (fill (color 0 0 0 0.0000))
-    (property "Sheetname" "Ethernet" (at 67.31 60.2484 0)
+    (property "Sheetname" "Power Supply" (at 78.105 111.0484 0)
       (effects (font (size 1.27 1.27)) (justify left bottom))
     )
-    (property "Sheetfile" "eth.kicad_sch" (at 67.31 89.4846 0)
+    (property "Sheetfile" "psu.kicad_sch" (at 78.105 116.1546 0)
+      (effects (font (size 1.27 1.27)) (justify left top))
+    )
+    (instances
+      (project "Node"
+        (path "/48ecc24b-1ca1-455a-ac86-9597a620a90f" (page "7"))
+      )
+    )
+  )
+  (sheet (at 78.105 53.975) (size 17.145 26.035) (fields_autoplaced)
+    (stroke (width 0.1524) (type solid))
+    (fill (color 0 0 0 0.0000))
+    (property "Sheetname" "Ethernet" (at 78.105 53.2634 0)
+      (effects (font (size 1.27 1.27)) (justify left bottom))
+    )
+    (property "Sheetfile" "eth.kicad_sch" (at 78.105 80.5946 0)
       (effects (font (size 1.27 1.27)) (justify left top))
     )
@@
     )
   )
-  (sheet (at 104.14 99.695) (size 30.48 27.94) (fields_autoplaced)
+  (sheet (at 78.105 86.995) (size 17.145 8.89) (fields_autoplaced)
     (stroke (width 0.1524) (type solid))
     (fill (color 0 0 0 0.0000))
-    (property "Sheetname" "Flash Interface" (at 104.14 98.9834 0)
+    (property "Sheetname" "Flash Interface" (at 78.105 86.2834 0)
       (effects (font (size 1.27 1.27)) (justify left bottom))
     )
-    (property "Sheetfile" "flash.kicad_sch" (at 104.14 128.2196 0)
+    (property "Sheetfile" "flash.kicad_sch" (at 78.105 96.4696 0)
       (effects (font (size 1.27 1.27)) (justify left top))
     )
@@
     )
   )
-  (sheet (at 110.49 53.975) (size 19.05 31.75) (fields_autoplaced)
+  (sheet (at 103.505 53.975) (size 26.035 51.435) (fields_autoplaced)
     (stroke (width 0.1524) (type solid))
     (fill (color 0 0 0 0.0000))
-    (property "Sheetname" "ESP32" (at 110.49 53.2634 0)
+    (property "Sheetname" "ESP32" (at 103.505 53.2634 0)
       (effects (font (size 1.27 1.27)) (justify left bottom))
     )
-    (property "Sheetfile" "esp32.kicad_sch" (at 110.49 86.3096 0)
+    (property "Sheetfile" "esp32.kicad_sch" (at 103.505 105.9946 0)
       (effects (font (size 1.27 1.27)) (justify left top))
+    )
+    (pin "EN" input (at 103.505 87.63 180)
+      (effects (font (size 1.27 1.27)) (justify left))
+    )
+    (pin "UART_TX0" input (at 103.505 91.44 180)
+      (effects (font (size 1.27 1.27)) (justify left))
+    )
+    (pin "UART_RX0" output (at 103.505 93.345 180)
+      (effects (font (size 1.27 1.27)) (justify left))
+    )
+    (pin "I2S_SCL" output (at 129.54 86.36 0)
+      (effects (font (size 1.27 1.27)) (justify right))
+    )
+    (pin "I2S0_WS" output (at 129.54 81.28 0)
+      (effects (font (size 1.27 1.27)) (justify right))
+    )
+    (pin "I2S1_DOUT" output (at 129.54 91.44 0)
+      (effects (font (size 1.27 1.27)) (justify right))
+    )
+    (pin "IO0" input (at 103.505 89.535 180)
+      (effects (font (size 1.27 1.27)) (justify left))
+    )
+    (pin "PHY_PWR" output (at 103.505 55.88 180)
+      (effects (font (size 1.27 1.27)) (justify left))
+    )
+    (pin "I2S1_WS" output (at 129.54 88.9 0)
+      (effects (font (size 1.27 1.27)) (justify right))
+    )
+    (pin "MDC(RMII)" output (at 103.505 71.12 180)
+      (effects (font (size 1.27 1.27)) (justify left))
+    )
+    (pin "EMAC_RX_CRX_DV" output (at 103.505 73.66 180)
+      (effects (font (size 1.27 1.27)) (justify left))
+    )
+    (pin "I2C_SCL" output (at 129.54 101.6 0)
+      (effects (font (size 1.27 1.27)) (justify right))
+    )
+    (pin "I2C_SDA" bidirectional (at 129.54 99.06 0)
+      (effects (font (size 1.27 1.27)) (justify right))
+    )
+    (pin "EMAC_RXD1(RMII)" output (at 103.505 63.5 180)
+      (effects (font (size 1.27 1.27)) (justify left))
+    )
+    (pin "EMAC_TXD1(RMII)" input (at 103.505 66.04 180)
+      (effects (font (size 1.27 1.27)) (justify left))
+    )
+    (pin "EMAC_RXD0(RMII)" output (at 103.505 58.42 180)
+      (effects (font (size 1.27 1.27)) (justify left))
+    )
+    (pin "I2S0_DOUT" output (at 129.54 83.82 0)
+      (effects (font (size 1.27 1.27)) (justify right))
+    )
+    (pin "MDIO(RMII)" bidirectional (at 103.505 76.2 180)
+      (effects (font (size 1.27 1.27)) (justify left))
+    )
+    (pin "EMAC_CLK_OUT_180" output (at 103.505 78.105 180)
+      (effects (font (size 1.27 1.27)) (justify left))
+    )
+    (pin "EMAC_TXD0(RMII)" input (at 103.505 60.96 180)
+      (effects (font (size 1.27 1.27)) (justify left))
+    )
+    (pin "EMAC_TX_EN(RMII)" output (at 103.505 68.58 180)
+      (effects (font (size 1.27 1.27)) (justify left))
     )
     (instances
@@
     )
   )
-  (sheet (at 167.64 67.945) (size 21.59 32.385) (fields_autoplaced)
+  (sheet (at 137.795 97.79) (size 19.685 5.08) (fields_autoplaced)
     (stroke (width 0.1524) (type solid))
     (fill (color 0 0 0 0.0000))
-    (property "Sheetname" "IO" (at 167.64 67.2334 0)
+    (property "Sheetname" "IO" (at 137.795 97.0784 0)
       (effects (font (size 1.27 1.27)) (justify left bottom))
     )
-    (property "Sheetfile" "io.kicad_sch" (at 167.64 100.9146 0)
+    (property "Sheetfile" "io.kicad_sch" (at 137.795 103.4546 0)
       (effects (font (size 1.27 1.27)) (justify left top))
     )
