File: Hardware/Node/esp32.kicad_sch (KiCad schematic)
At the start: 4 parts, among them U1 ESP32-WROOM-32UE_(16MB)

Commit message: Updated schematic
Parts:
- added D1: WS2812B-2020, manul_tech:LED_WS2812C-2020, symbol manul_tech:WS2812B-2020
Connections:
- net +3.3V: now also D1.4 (VDD)
- net GND: now also D1.2 (GND)
- net USR_LED: now reaches U1.26 (IO4)
- net USR_LED: now also D1.3 (DIN)
- net I2C_SCL: now reaches U1.8 (IO32)
- net I2C_SDA: now reaches U1.9 (IO33)
- no-connect marks 2 -> 6
Changed lines of the file:
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@@
   (junction (at 101.6 57.15) (diameter 0) (color 0 0 0 0)
   )
+  (no_connect (at 125.73 77.47))
+  (no_connect (at 125.73 74.93))
+  (no_connect (at 235.585 62.23))
   (no_connect (at 125.73 64.77))
+  (no_connect (at 166.37 59.69))
   (no_connect (at 125.73 67.31))
   (wire (pts (xy 166.37 80.01) (xy 193.04 80.01))
@@
     (stroke (width 0) (type default))
   )
-  (wire (pts (xy 166.37 62.23) (xy 193.04 62.23))
+  (wire (pts (xy 166.37 62.23) (xy 220.345 62.23))
     (stroke (width 0) (type default))
   )
@@
     (stroke (width 0) (type default))
   )
-  (wire (pts (xy 166.37 59.69) (xy 193.04 59.69))
-    (stroke (width 0) (type default))
-  )
   (wire (pts (xy 166.37 102.87) (xy 193.04 102.87))
     (stroke (width 0) (type default))
+  )
+  (label "USR_LED" (at 193.04 62.23 180) (fields_autoplaced)
+    (effects (font (size 1.27 1.27)) (justify right bottom))
   )
   (hierarchical_label "MDC(RMII)" (shape output) (at 193.04 92.71 0) (fields_autoplaced)
@@
     (effects (font (size 1.27 1.27)) (justify left))
   )
-  (hierarchical_label "I2S0_DOUT" (shape bidirectional) (at 193.04 77.47 0) (fields_autoplaced)
+  (hierarchical_label "I2S0_DOUT" (shape output) (at 193.04 77.47 0) (fields_autoplaced)
     (effects (font (size 1.27 1.27)) (justify left))
   )
@@
     (effects (font (size 1.27 1.27)) (justify right))
   )
+  (hierarchical_label "I2C_SDA" (shape bidirectional) (at 193.04 105.41 0) (fields_autoplaced)
+    (effects (font (size 1.27 1.27)) (justify left))
+  )
   (hierarchical_label "MDIO(RMII)" (shape bidirectional) (at 193.04 82.55 0) (fields_autoplaced)
     (effects (font (size 1.27 1.27)) (justify left))
   )
+  (hierarchical_label "I2C_SCL" (shape output) (at 193.04 102.87 0) (fields_autoplaced)
+    (effects (font (size 1.27 1.27)) (justify left))
+  )
   (hierarchical_label "I2S1_WS" (shape output) (at 193.04 67.31 0) (fields_autoplaced)
     (effects (font (size 1.27 1.27)) (justify left))
@@
     (effects (font (size 1.27 1.27)) (justify left))
   )
-  (hierarchical_label "I2S1_DOUT" (shape bidirectional) (at 193.04 69.85 0) (fields_autoplaced)
+  (hierarchical_label "I2S1_DOUT" (shape output) (at 193.04 69.85 0) (fields_autoplaced)
     (effects (font (size 1.27 1.27)) (justify left))
   )
@@
         (path "/48ecc24b-1ca1-455a-ac86-9597a620a90f/a5545c38-9a32-4b82-a707-3d96a31e434d"
           (reference "C2") (unit 1)
+        )
+      )
+    )
+  )
+  (symbol (lib_id "manul_tech:WS2812B-2020") (at 227.965 62.23 0) (unit 1)
+    (in_bom yes) (on_board yes) (dnp no) (fields_autoplaced)
+    (property "Reference" "D1" (at 241.4681 57.0339 0)
+      (effects (font (size 1.27 1.27)))
+    )
+    (property "Value" "WS2812B-2020" (at 241.4681 59.0819 0)
+      (effects (font (size 1.27 1.27)))
+    )
+    (property "Footprint" "manul_tech:LED_WS2812C-2020" (at 233.045 71.12 0)
+      (effects (font (size 1.27 1.27)) (justify left top) hide)
+    )
+    (property "Datasheet" "" (at 218.44 64.77 90)
+      (effects (font (size 1.27 1.27)) (justify left top) hide)
+    )
+    (property "internalRef" "8.02.003" (at 241.4681 61.1299 0)
+      (effects (font (size 1.27 1.27)))
+    )
+    (pin "1")
+    (pin "2")
+    (pin "3")
+    (pin "4")
+    (instances
+      (project "Node"
+        (path "/48ecc24b-1ca1-455a-ac86-9597a620a90f/a5545c38-9a32-4b82-a707-3d96a31e434d"
+          (reference "D1") (unit 1)
+        )
+      )
+    )
+  )
+  (symbol (lib_id "power:GND") (at 227.965 69.85 0) (unit 1)
+    (in_bom yes) (on_board yes) (dnp no) (fields_autoplaced)
+    (property "Reference" "#PWR07" (at 227.965 76.2 0)
+      (effects (font (size 1.27 1.27)) hide)
+    )
+    (property "Value" "GND" (at 227.965 73.795 0)
+      (effects (font (size 1.27 1.27)))
+    )
+    (property "Footprint" "" (at 227.965 69.85 0)
+      (effects (font (size 1.27 1.27)) hide)
+    )
+    (property "Datasheet" "" (at 227.965 69.85 0)
+      (effects (font (size 1.27 1.27)) hide)
+    )
+    (pin "1")
+    (instances
+      (project "Node"
+        (path "/48ecc24b-1ca1-455a-ac86-9597a620a90f/a5545c38-9a32-4b82-a707-3d96a31e434d"
+          (reference "#PWR07") (unit 1)
         )
       )
@@
         )
       )
+    )
+  )
+  (symbol (lib_id "power:+3.3V") (at 227.965 54.61 0) (unit 1)
+    (in_bom yes) (on_board yes) (dnp no) (fields_autoplaced)
+    (property "Reference" "#PWR06" (at 227.965 58.42 0)
+      (effects (font (size 1.27 1.27)) hide)
+    )
+    (property "Value" "+3.3V" (at 227.965 50.665 0)
+      (effects (font (size 1.27 1.27)))
+    )
+    (property "Footprint" "" (at 227.965 54.61 0)
+      (effects (font (size 1.27 1.27)) hide)
+    )
+    (property "Datasheet" "" (at 227.965 54.61 0)
+      (effects (font (size 1.27 1.27)) hide)
+    )
+    (pin "1")
+    (instances
+      (project "Node"
+        (path "/48ecc24b-1ca1-455a-ac86-9597a620a90f/a5545c38-9a32-4b82-a707-3d96a31e434d"
+          (reference "#PWR06") (unit 1)
+        )
+      )
